File: p48_pip_adapter.kicad_sch (KiCad schematic)
At the start: 20 parts, among them J1 XLR3, Q1 MMBT3904, Q2 MMBT3906, Q3 MMBT3906

Commit message: Add board-on-connector render and schematic to the README
- images/board_with_connector.png: the routed board (kicad-cli GLB) plugged
  into a bare 3-pin XLR insert, rendered in Blender. Reproduced by
  scripts/render_connector.py (+ render_connector_blender.py, tmf2stl.py); the
  connector model is third-party and kept local/gitignored (reference/).
- images/schematic.png: exported from the wired schematic for expert review.
  Schematic paper A4 -> A3 (components no longer overflow the sheet) and a
  title block added.

Co-Authored-By: Claude Opus 4.8 (1M context) <noreply@anthropic.com>
Other:
- company: (none) -> github.com/tphakala/p48-pip-adapter
- title: (none) -> P48 to 8V PIP Adapter
Changed lines of the file:
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@@
 (kicad_sch (version 20230121) (generator eeschema)
-  (paper "A4")
+  (paper "A3")
+  (title_block
+    (title "P48 to 8V PIP Adapter")
+    (rev "A")
+    (company "github.com/tphakala/p48-pip-adapter")
+    (comment 1 "Impedance-balanced phantom-power to plug-in-power mic adapter")
+    (comment 2 "Connectivity by net labels; see netlist.py / SPEC.md for the authoritative net list")
+  )
   (symbol (lib_id "Connector:XLR3") (at 40 45 0) (unit 1)
     (in_bom yes) (on_board yes) (dnp no)
